File: pcb/simpleCH552.brd (EAGLE design)
At the start: 40.6 x 12 mm, 16 parts, among them U2 CH552G, X1 USBPCB

Commit message: Update simpleCH552.brd
Routing:
- net N$1: track 16.4 -> 19.1 mm
- net +5V: track 72.1 -> 71.5 mm
Changed lines of the file:
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@@
 <wire x1="28.4769125" y1="8.27243125" x2="28.9052" y2="7.84414375" width="0.2032" layer="16"/>
 <wire x1="28.9052" y1="7.1628" x2="28.9052" y2="7.84414375" width="0.2032" layer="16"/>
-<wire x1="32.7" y1="10.5664" x2="32.7" y2="10.0736" width="0.2032" layer="1"/>
-<wire x1="32.7" y1="10.0736" x2="34.2646" y2="8.509" width="0.2032" layer="1"/>
+<wire x1="32.7" y1="10.0736" x2="32.7914" y2="9.9822" width="0.2032" layer="1"/>
 <via x="29.4526875" y="5.0178875" extent="1-16" drill="0.35"/>
-<wire x1="34.2646" y1="8.509" x2="34.6964" y2="8.0772" width="0.2032" layer="1"/>
+<wire x1="32.7914" y1="9.9822" x2="34.6964" y2="8.0772" width="0.2032" layer="1"/>
 <wire x1="29.4526875" y1="5.0178875" x2="29.746175" y2="4.7244" width="0.2032" layer="1"/>
 <wire x1="29.746175" y1="4.7244" x2="33.4772" y2="4.7244" width="0.2032" layer="1"/>
@@
 <wire x1="29.5656" y1="5.334" x2="29.5656" y2="6.5024" width="0.2032" layer="16"/>
 <wire x1="29.5656" y1="6.5024" x2="28.9052" y2="7.1628" width="0.2032" layer="16"/>
-<wire x1="34.2646" y1="8.509" x2="39.0398" y2="8.509" width="0.2032" layer="1"/>
-<wire x1="39.461" y1="8.0878" x2="39.461" y2="2.0194" width="0.2032" layer="1"/>
-<wire x1="39.0398" y1="8.509" x2="39.461" y2="8.0878" width="0.2032" layer="1"/>
-<wire x1="39.461" y1="2.0194" x2="39.461" y2="2.195" width="0.2032" layer="1"/>
-<wire x1="39.461" y1="2.195" x2="38.1" y2="3.5052" width="0.2032" layer="1"/>
-<wire x1="38.1" y1="3.5052" x2="38.1" y2="7.5184" width="1.27" layer="1"/>
+<wire x1="39.461" y1="2.0194" x2="39.461" y2="2.136615625" width="0.2032" layer="1"/>
+<wire x1="39.461" y1="2.136615625" x2="38.2524" y2="3.3001" width="0.2032" layer="1"/>
+<wire x1="38.2524" y1="3.3001" x2="38.2016" y2="3.349003125" width="0.2032" layer="1"/>
+<wire x1="38.2524" y1="8.5344" x2="38.2524" y2="3.3001" width="1.27" layer="1"/>
+<wire x1="32.7" y1="10.5664" x2="33.3096" y2="11.176" width="0.2032" layer="1"/>
+<wire x1="33.3096" y1="11.176" x2="37.5412" y2="11.176" width="0.2032" layer="1"/>
+<wire x1="37.9476" y1="10.1092" x2="37.9476" y2="8.5344" width="1.27" layer="1"/>
+<wire x1="38.2524" y1="8.5344" x2="37.9476" y2="8.5344" width="0.2032" layer="1"/>
+<wire x1="38.2016" y1="3.349003125" x2="38.2016" y2="3.2512" width="0.2032" layer="1"/>
+<wire x1="38.0492" y1="3.0988" x2="38.0492" y2="1.9304" width="1.27" layer="1"/>
+<wire x1="38.2016" y1="3.2512" x2="38.0492" y2="3.0988" width="0.2032" layer="1"/>
+<wire x1="37.5412" y1="11.176" x2="37.9476" y2="10.7696" width="0.2032" layer="1"/>
+<wire x1="37.9476" y1="10.7696" x2="37.9476" y2="10.1092" width="0.2032" layer="1"/>
+<wire x1="32.7" y1="10.5664" x2="32.7914" y2="10.475" width="0.2032" layer="1"/>
+<wire x1="32.7914" y1="10.475" x2="32.7914" y2="9.9822" width="0.2032" layer="1"/>
 </signal>
 <signal name="P1.4">
@@
 <wire x1="33.02" y1="5.6896" x2="33.02" y2="3.1496" width="0.2032" layer="16"/>
 <wire x1="33.02" y1="3.1496" x2="34.1884" y2="1.9812" width="0.2032" layer="16"/>
-<wire x1="34.961" y1="2.0194" x2="36.322" y2="3.5052" width="0.2032" layer="1"/>
-<wire x1="36.322" y1="3.5052" x2="36.322" y2="7.5184" width="1.27" layer="1"/>
+<wire x1="36.1696" y1="8.5344" x2="36.1696" y2="3.338825" width="1.27" layer="1"/>
+<wire x1="36.1696" y1="8.5344" x2="36.4744" y2="8.5344" width="0.2032" layer="1"/>
+<wire x1="36.4744" y1="8.5344" x2="36.4744" y2="10.1092" width="1.27" layer="1"/>
+<wire x1="36.1696" y1="3.338825" x2="36.4236" y2="3.084825" width="0.2032" layer="1"/>
+<wire x1="36.4236" y1="1.9304" x2="36.4236" y2="3.084825" width="1.27" layer="1"/>
+<wire x1="36.322" y1="1.9812" x2="36.3728" y2="1.9812" width="0.2032" layer="1"/>
+<wire x1="36.3728" y1="1.9812" x2="36.4236" y2="1.9304" width="0.2032" layer="1"/>
 </signal>
 <signal name="N$3">
